File: kicad/ADF Board/MW_Source.kicad_sch (KiCad schematic)
At the start: 126 parts, among them IC3 ADF4351BCPZ, IC4 LTC5589IUF#PBF, J10 Conn_Coaxial, J11 Conn_Coaxial, J18 Conn_Coaxial, J2 Conn_Coaxial, U12 GRF2012, U2 AD8137, U8 M3SWA2-63DRC, U9 GRF2012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

Commit message: Started parts selection for assemblability Considering deleting the I/Q modulator and periphery
Parts:
- added C301: 10n, symbol Device:C_Small
- D6, D7: value SZMMSZ5232BT1G -> BZT52C5V6; LCSC (none) -> C19077402
- R11, R12: now not fitted
- Y2: value TG2520SMN_30.000M-MCGNNM0 -> 30MHz_3Y030000VP; LCSC (none) -> C22370490
Connections:
- net GND: now also C301.2
- net at C75.1, C77.1, FB2.1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: now also C301.1
Other:
- moved on the sheet: C75, C77

Commit message: Deleted I/Q mod, switch, charge pump Found candidates for RF amp and PLL
Parts:
- removed C120, C69, C76, C78, C79, C81: 100n, Capacitor_SMD:C_0603_1608Metric, symbol Device:C
- removed C130: 1u, Capacitor_SMD:C_0603_1608Metric, symbol Device:C
- removed C56: 4.7u, Capacitor_SMD:C_0805_2012Metric, symbol Device:C
- removed C58, C62: 1n, Capacitor_SMD:C_0603_1608Metric, symbol Device:C
- removed C6, C7: 0.1u, Capacitor_SMD:C_0603_1608Metric, symbol Device:C
- removed C70, C85: 0.2p, Capacitor_SMD:C_0402_1005Metric, symbol Device:C
- removed C73: 2p, Capacitor_SMD:C_0402_1005Metric, symbol Device:C
- removed C8, C9: 10n, Capacitor_SMD:C_0603_1608Metric, symbol Device:C
- removed C83: DNI, Capacitor_SMD:C_0603_1608Metric, symbol Device:C
- removed C84, C93: 100p, Capacitor_SMD:C_0402_1005Metric, symbol Device:C
- removed C87, C88: 1p, Capacitor_SMD:C_0402_1005Metric, symbol Device:C
- removed C90, C91: 0.5p, Capacitor_SMD:C_0402_1005Metric, symbol Device:C
- removed D4: 1N4148, Diode_SMD:D_SOD-123, symbol Diode:1N4148
- removed D6, D7: BZT52C5V6, Diode_SMD:D_SOD-123, symbol Device:D_Zener
- removed FB1: MPZ1608S331AT, Inductor_SMD:L_0603_1608Metric, symbol Device:FerriteBead
- removed IC4: LTC5589IUF#PBF, SamacSys_Parts:QFN50P400X400X80-25N-D, symbol SamacSys_Parts:LTC5589IUF#PBF
- removed J2: Conn_Coaxial, Connector_Coaxial:U.FL_Hirose_U.FL-R-SMT-1_Vertical, symbol Connector:Conn_Coaxial
- removed JP11: Jumper_2_Bridged, Jumper:SolderJumper-2_P1.3mm_Open_RoundedPad1.0x1.5mm, symbol Jumper:Jumper_2_Bridged
- removed JP4, JP5, JP6: SolderJumper_2_Open, Jumper:SolderJumper-2_P1.3mm_Open_RoundedPad1.0x1.5mm, symbol Jumper:SolderJumper_2_Open
- removed L9: 4.7n, Inductor_SMD:L_0402_1005Metric, symbol Device:L
- removed R10, R7, R8, R9: 10k, Capacitor_SMD:C_0603_1608Metric, symbol Device:R
- removed R11, R12: R, Resistor_SMD:R_0603_1608Metric, symbol Device:R
- removed R13: 1.15k, Resistor_SMD:R_0603_1608Metric, symbol Device:R
- removed R14: 500, Resistor_SMD:R_0603_1608Metric, symbol Device:R
- removed R49, R70: 1k, Resistor_SMD:R_0603_1608Metric, symbol Device:R
- removed R53: 100k, Resistor_SMD:R_0603_1608Metric, symbol Device:R
- removed R6: 50, Resistor_SMD:R_0402_1005Metric, symbol Device:R
- removed R60: 1R, Resistor_SMD:R_0603_1608Metric, symbol Device:R
- removed R62, R76, R78, R79: DNI, Resistor_SMD:R_0603_1608Metric, symbol Device:R
- removed R63: 0R, Resistor_SMD:R_0603_1608Metric, symbol Device:R
- removed R65, R68, R71, R72: 49.9R, Resistor_SMD:R_0603_1608Metric, symbol Device:R
- removed R77: 10R, Resistor_SMD:R_0603_1608Metric, symbol Device:R
- removed R80: 100R, Resistor_SMD:R_0402_1005Metric, symbol Device:R
- removed R81, R82: 11.5R, Resistor_SMD:R_0402_1005Metric, symbol Device:R
- removed TP23: IQ_Vctrl, TestPoint:TestPoint_Pad_D2.0mm, symbol Connector:TestPoint
- removed TP26: IQ_EN, TestPoint:TestPoint_Pad_D2.0mm, symbol Connector:TestPoint
- removed TP31: IQ_SDO2, TestPoint:TestPoint_Pad_D2.0mm, symbol Connector:TestPoint
- removed TP7: IQ_TTCK, TestPoint:TestPoint_Pad_D2.0mm, symbol Connector:TestPoint
- removed U2: AD8137, Package_SO:SOIC-8_3.9x4.9mm_P1.27mm, symbol Amplifier_Operational:LTC6362xMS8
- removed U8: M3SWA2-63DRC, Package_DFN_QFN:QFN-12-1EP_3x3mm_P0.51mm_EP1.45x1.45mm, symbol parts:M3SWA2-63DRC
- IC3: value ADF4351BCPZ -> ADF4350BCPZ-RL7; LCSC (none) -> C98705; Manufacturer_Name Analog Devices -> (none); Manufacturer_Part_Number ADF4351BCPZ -> (none); Mouser Part Number 584-ADF4351BCPZ -> (none); Mouser Price/Stock https://www.mouser.co.uk/ProductDetail/Analog-Devices/ADF43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 -> (none)
Connections:
- net Switch1_Out is gone; now on net PLL_Out: U9.3 (IN)
Other:
- note added: "ADF4351 was originally designed, but ADF4350 has more stock."
- note added: "Netlabel bush"
- note added: "TODO replace for parts in stock"
- note removed: "1,4V"
- note removed: "1V max."
- note removed: "HF-Switch"
- note removed: "IQ Modulator"
- note removed: "Power consumption +-45mW (90mW total)"
- note removed: "Power consumption 132mW"
- note removed: "Single ended to differential driver for IQ Modulator Imi/Ipi"

Commit message: Finished part selection and rearranged schematic
Parts:
- removed C103, C115: 1000p, Capacitor_SMD:C_0402_1005Metric, symbol Device:C
- removed C110, C98: 0.1u, Capacitor_SMD:C_0402_1005Metric, symbol Device:C
- removed C119: 100n, Capacitor_SMD:C_0603_1608Metric, symbol Device:C
- removed C129: 1u, Capacitor_SMD:C_0603_1608Metric, symbol Device:C
- removed C75: 0.1u, Capacitor_SMD:C_0603_1608Metric, symbol Device:C
- removed L10, L11: 47n, Inductor_SMD:L_0603_1608Metric, symbol Device:L
- removed R5, R91: 0R, Capacitor_SMD:C_0402_1005Metric, symbol Device:R
- removed R89, R93: 250R, Capacitor_SMD:C_0402_1005Metric, symbol Device:R
- removed U12, U9: GRF2012, Package_DFN_QFN:DFN-6-1EP_2x2mm_P0.5mm_EP0.6x1.37mm, symbol parts:GRF2012
- C101, C60, C61, C68, C74, C92, C95, C96: value 0.1u -> 100n; LCSC (none) -> C14663
- C104, C105, C106, C114, C57, C63, C71: LCSC (none) -> C1634
- C301: footprint (none) -> Capacitor_SMD:C_0402_1005Metric; LCSC (none) -> C15195
- C50: value 10p -> 10p/C0G/50V; LCSC (none) -> C32949
- C51, C52: value 0.7p -> 0.7p/C0G/50V; LCSC (none) -> C397301
- C53: value 1.2n -> 1.5n; LCSC (none) -> C1595
- C54: LCSC (none) -> C107091
- C55: LCSC (none) -> C1609
- C77: footprint Capacitor_SMD:C_0603_1608Metric -> Capacitor_SMD:C_0805_2012Metric; LCSC (none) -> C28323
- C80, C82: LCSC (none) -> C1523
- D5: value LED -> yellow_PLL-lock; footprint LED_SMD:LED_0805_2012Metric -> LED_SMD:LED_0603_1608Metric; LCSC (none) -> C72038
- FB2: value MPZ1608S331AT -> GZ1608D601TF; LCSC (none) -> C1002
- J10: value Conn_Coaxial -> IPEX/U.FL_PLL_out_RFBP; LCSC (none) -> C496552
- J11: value Conn_Coaxial -> IPEX/U.FL_PLL-ref-in; LCSC (none) -> C496552
- J18: value Conn_Coaxial -> IPEX/U.FL_PLL_out_RFBN; LCSC (none) -> C496552
- L6, L7: value 3.3n -> 3.3nH; LCSC (none) -> C3223325
- L8: value 10n -> 10nH; LCSC (none) -> C382409
- R44: LCSC (none) -> C23228
- R45, R75: LCSC (none) -> C21189
- R46: LCSC (none) -> C25194
- R47: now not fitted
- R50: LCSC (none) -> C21190
- R55: LCSC (none) -> C22775
- R57: LCSC (none) -> C23162
- R66: value 750R -> 1k; LCSC (none) -> C21190
- R73: LCSC (none) -> C23185
Connections:
- net +3.3V: now also L8.2; no longer L8.1
- net at C52.1, IC3.13 (RFOUTA-), L6.2: now also L8.1; no longer L8.2
- net SCKL renamed SCK
Other:
- note added: "ADF4351 was originally designed, but ADF4350 has more stock. Is pin-compatible and is register-compatible for almost all functions."
- note added: "Aux outputs of PLL chip"
- note added: "Balun as specified in datasheet for requency range 1600 to 3600 MHz. PLL_Out controlled 50R impedance."
- note added: "HI when PLL lock 2.9V min."
- note added: "Power consumption: 0.558W 170mA@3.3V"
- note added: "RF inductor multilayer ceramic 10nH 2% Q min. 8 DCR 0.29R@0.2A SRF 3.2GHz"
- note added: "RF inductor wire-wound chip 3.3nH 6% Q min. 30 DCR 0.040R@0.9A SRF 12GHz"
- note added: "U.FL is the same as I-PEX, IPX, and UMCC. JLC calls them IPEX"
- note added: "at pin 26"
- note added: "non-standard capacitance values from datasheet example"
- note added: "originally 330R@100MHz DC 0.08R@1.7A exact value doesn't matter now 600R@100MHz DC 0.45R@0.2A"
- note added: "target 1 mA @ 2V"
- note added: "target 1.2nF"
- note removed: "ADF4351 was originally designed, but ADF4350 has more stock."
- note removed: "Die passiven Bauteile, die ich ab dem PLL Ausgang im Mikrowellenpfad verwendetet habe, sind mit Mouser Links hinterlegt."
- note removed: "Gain Stage +28dB"
- note removed: "Netlabel bush"
- note removed: "Power consumption: 0.558W"
- note removed: "TODO replace for parts in stock"
- moved on the sheet: C101, C104, C105, C106, C114, C301, C50, C51, C52, C53, C54, C55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
