File: kicad/ADF Board/MW_Source.kicad_sch (KiCad schematic)
At the start: 45 parts, among them IC3 ADF4350BCPZ-RL7, J10 IPEX/U.FL_PLL_out_RFBP, J11 IPEX/U.FL_PLL-ref-in, J18 IPEX/U.FL_PLL_out_RFBN, Y2 30MHz_3Y030000VP

Commit message: Finished board, DRC OK, silkscreen done, sheets versioned. Ready for export.
Parts:
- renumbered C50 to C401, C51 to C402, C101 to C403, C52 to C404, C114 to C405, C96 to C406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
Other:
- company: (none) -> openUC2 GmbH
- title: (none) -> QuantumMiniLabs_ODMR::ADF_Board
