File: kicad/ADF Board/ADF_Board.kicad_sch (KiCad schematic)
At the start: 5 parts, among them J3 SMA-elbowed_to-NV-diamonds

Commit message: Finished board, DRC OK, silkscreen done, sheets versioned. Ready for export.
Parts:
- removed H104: M3, MountingHole:MountingHole_3.2mm_M3_Pad_Via, symbol Mechanical:MountingHole_Pad
- renumbered J3 to J101
Other:
- company: (none) -> openUC2 GmbH
- title: (none) -> QuantumMiniLabs_ODMR::ADF_Board
Changed lines of the file:
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@@
 	(generator_version "9.0")
 	(paper "A4")
+	(title_block
+		(title "QuantumMiniLabs_ODMR::ADF_Board")
+		(date "2025-03-01")
+		(rev "A")
+		(company "openUC2 GmbH")
+		(comment 1 "christiankuttke based on design by Dennis Stiegekötter")
+	)
 	(text "HF netclass traces need impedance matching to 50 Ohm!\nUse JLC impedance calculator with controlled stackup to determine trace width.\nSingle Ended Non Coplanar"
 		(exclude_from_sim no)
@@
 		(color 0 0 0 0)
 	)
-	(junction
-		(at 63.5 120.65)
-		(diameter 0)
-		(color 0 0 0 0)
-	)
 	(no_connect
 		(at 55.88 39.37)
@@
 	(wire
 		(pts
-			(xy 63.5 114.3) (xy 63.5 120.65)
+			(xy 63.5 114.3) (xy 63.5 127)
 		)
 		(stroke
@@
 		(pts
 			(xy 99.06 41.91) (xy 99.06 31.75)
-		)
-		(stroke
-			(width 0)
-			(type default)
-		)
-	)
-	(wire
-		(pts
-			(xy 63.5 120.65) (xy 63.5 127)
 		)
 		(stroke
@@
 		(dnp no)
 		(fields_autoplaced yes)
-		(property "Reference" "J3"
+		(property "Reference" "J101"
 			(at 243.84 47.2833 0)
 			(effects
@@
 			(project ""
 				(path "/90b3de2f-c818-48df-8078-fde6a4536a1f"
-					(reference "J3")
+					(reference "J101")
 					(unit 1)
 				)
@@
 		(dnp no)
 		(fields_autoplaced yes)
-		(property "Reference" "#PWR0127"
+		(property "Reference" "#PWR0101"
 			(at 63.5 133.35 0)
 			(effects
@@
 			(project ""
 				(path "/90b3de2f-c818-48df-8078-fde6a4536a1f"
-					(reference "#PWR0127")
-					(unit 1)
-				)
-			)
-		)
-	)
-	(symbol
-		(lib_id "Mechanical:MountingHole_Pad")
-		(at 66.04 120.65 270)
-		(unit 1)
-		(exclude_from_sim yes)
-		(in_bom no)
-		(on_board yes)
-		(dnp no)
-		(fields_autoplaced yes)
-		(property "Reference" "H104"
-			(at 69.85 119.3799 90)
-			(effects
-				(font
-					(size 1.27 1.27)
-				)
-				(justify left)
-			)
-		)
-		(property "Value" "M3"
-			(at 69.85 121.9199 90)
-			(effects
-				(font
-					(size 1.27 1.27)
-				)
-				(justify left)
-			)
-		)
-		(property "Footprint" "MountingHole:MountingHole_3.2mm_M3_Pad_Via"
-			(at 66.04 120.65 0)
-			(effects
-				(font
-					(size 1.27 1.27)
-				)
-				(hide yes)
-			)
-		)
-		(property "Datasheet" "~"
-			(at 66.04 120.65 0)
-			(effects
-				(font
-					(size 1.27 1.27)
-				)
-				(hide yes)
-			)
-		)
-		(property "Description" "Mounting Hole with connection"
-			(at 66.04 120.65 0)
-			(effects
-				(font
-					(size 1.27 1.27)
-				)
-				(hide yes)
-			)
-		)
-		(property "Description_1" ""
-			(at 66.04 120.65 0)
-			(effects
-				(font
-					(size 1.27 1.27)
-				)
-				(hide yes)
-			)
-		)
-		(pin "1"
-		)
-		(instances
-			(project "ADF_Board"
-				(path "/90b3de2f-c818-48df-8078-fde6a4536a1f"
-					(reference "H104")
+					(reference "#PWR0101")
 					(unit 1)
 				)
@@
 		(at 66.04 114.3 270)
 		(unit 1)
-		(exclude_from_sim yes)
+		(exclude_from_sim no)
 		(in_bom no)
 		(on_board yes)
@@
 		(dnp no)
 		(fields_autoplaced yes)
-		(property "Reference" "#PWR0101"
+		(property "Reference" "#PWR0102"
 			(at 241.3 57.15 0)
 			(effects
@@
 			(project ""
 				(path "/90b3de2f-c818-48df-8078-fde6a4536a1f"
-					(reference "#PWR0101")
+					(reference "#PWR0102")
 					(unit 1)
 				)
@@
 		(at 66.04 107.95 270)
 		(unit 1)
-		(exclude_from_sim yes)
+		(exclude_from_sim no)
 		(in_bom no)
 		(on_board yes)
@@
 		(at 66.04 101.6 270)
 		(unit 1)
-		(exclude_from_sim yes)
+		(exclude_from_sim no)
 		(in_bom no)
 		(on_board yes)
