File: kicad/antenna-with-diamonds/antenna-with-diamonds.kicad_sch (KiCad schematic)
At the start: 2 parts, among them J101 SMA-elbowed_amplified-RF-input

Commit message: Finished silkscreen of antenna
Other:
- company: (none) -> openUC2 GmbH
- title: (none) -> QuantumMiniLabs_ODMR::antenna-with-diamonds
Changed lines of the file:
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@@
 	(generator_version "9.0")
 	(paper "A4")
+	(title_block
+		(title "QuantumMiniLabs_ODMR::antenna-with-diamonds")
+		(date "2025-09-22")
+		(rev "A")
+		(company "openUC2 GmbH")
+		(comment 1 "christiankuttke")
+	)
 	(text "3 NV-center Diamonds here, with 3-5 mm distance from each other"
 		(exclude_from_sim no)
